File: electronics_v02---smt/electronics_v02---smt.kicad_sch (KiCad schematic)
At the start: 24 parts, among them IC1 SN74HCT245PWR, IC2 MAX3485EESA+T, J1 171857-0004, J2 171857-0004, J3 171857-0003, J4 171857-0002, U1 RPiPicoW

Commit message: Add files via upload
Parts:
- added H1, H2: MountingHole, MountingHole:MountingHole_2.5mm, symbol Mechanical:MountingHole
- C1, C2: LCSC Part # (none) -> C1525; LCSC Part Number (none) -> C1525
- IC1: LCSC Part # (none) -> C6779; LCSC Part Number (none) -> C6779
- IC2: LCSC Part # (none) -> C9943; LCSC Part Number (none) -> C9943
- R1, R2, R3, R4: LCSC Part # (none) -> C15401; LCSC Part Number (none) -> C15401
- R10, R11, R12, R13, R6, R7, R8, R9: LCSC Part # (none) -> C25270; LCSC Part Number (none) -> C25270
- R14, R5: LCSC Part # (none) -> C4328; LCSC Part Number (none) -> C4328
Connections:
- net LED_1: now also J1.1; no longer J1.4
- net LED_2: now also J1.2; no longer J1.3
- net LED_3: now also J1.3; no longer J1.2
- net LED_4: now also J1.4; no longer J1.1
- net LED_5: now also J2.1; no longer J2.4
- net LED_6: now also J2.2; no longer J2.3
- net LED_7: now also J2.3; no longer J2.2
- net LED_8: now also J2.4; no longer J2.1
